Commit message: "Add gazebo sim"

File: src/robot_description/urdf/_robot.urdf.xacro (robot description, xacro)
@@ -3,3 +3,4 @@
     <xacro:include filename="_common.xacro" />
     <xacro:include filename="arm.xacro" />
+    <xacro:include filename="arm_gazebo.xacro" />
 </robot>

File: src/robot_description/urdf/arm.xacro (robot description, xacro)
@@ -1,13 +1,13 @@
 <?xml version="1.0" encoding="utf-8"?>
-<!-- <robot name="piper_arm" xmlns:xacro="http://www.ros.org/wiki/xacro"> -->
 <robot  xmlns:xacro="http://www.ros.org/wiki/xacro" >
     <!-- MESHES -->
-    <xacro:property name="arm_base_link" value="package://robot_description/meshes/arm_base_link.STL" />
-    <xacro:property name="arm_link1"     value="package://robot_description/meshes/arm_link1.STL" />
-    <xacro:property name="arm_link2"     value="package://robot_description/meshes/arm_link2.STL" />
-    <xacro:property name="arm_link3"     value="package://robot_description/meshes/arm_link3.STL" />
-    <xacro:property name="arm_link4"     value="package://robot_description/meshes/arm_link4.STL" />
-    <xacro:property name="arm_link5"     value="package://robot_description/meshes/arm_link5.STL" />
-    <xacro:property name="arm_link6"     value="package://robot_description/meshes/arm_link6.STL" />
+    <xacro:property name="mesh_path" value="file://$(find robot_description)/meshes" />
+    <xacro:property name="arm_base_link" value="${mesh_path}/arm_base_link.STL" />
+    <xacro:property name="arm_link1"     value="${mesh_path}/arm_link1.STL" />
+    <xacro:property name="arm_link2"     value="${mesh_path}/arm_link2.STL" />
+    <xacro:property name="arm_link3"     value="${mesh_path}/arm_link3.STL" />
+    <xacro:property name="arm_link4"     value="${mesh_path}/arm_link4.STL" />
+    <xacro:property name="arm_link5"     value="${mesh_path}/arm_link5.STL" />
+    <xacro:property name="arm_link6"     value="${mesh_path}/arm_link6.STL" />
     <!-- LINKS -->
     <!-- Link base -->
@@ -15,5 +15,6 @@
         <inertial>
             <origin xyz="-0.00473641164191482 2.56829134630247E-05 0.041451518036016" rpy="0 0 0"/>
-            <mass value="1.02"/>
+            <!-- <mass value="1.02"/> -->
+            <mass value="10.0"/>
             <inertia ixx="0.00267433" ixy="-0.00000073" ixz="-0.00017389"
                      iyy="0.00282612" iyz="0.0000004"   izz="0.00089624"/>

File: src/robot_moveit_config/config/piper_arm.ros2_control.xacro (robot description, xacro)
@@ -6,5 +6,6 @@
             <hardware>
                 <!-- By default, set up controllers for simulation. This won't work on real hardware -->
-                <plugin>mock_components/GenericSystem</plugin>
+                <!-- <plugin>mock_components/GenericSystem</plugin> -->
+                <plugin>gz_ros2_control/GazeboSimSystem</plugin>
             </hardware>
             <joint name="joint1">
@@ -51,4 +52,10 @@
             </joint>
         </ros2_control>
+        <gazebo>
+            <plugin filename="gz_ros2_control-system"
+                    name="gz_ros2_control::GazeboSimROS2ControlPlugin">
+                <parameters>$(find robot_moveit_config)/config/ros2_controllers.yaml</parameters>
+            </plugin>
+        </gazebo>
     </xacro:macro>
 </robot>

Commit message: Add motion tasks section

File: src/robot_description/urdf/_robot.urdf.xacro (robot description, xacro)
@@ -5,3 +5,4 @@
     <xacro:include filename="arm_gazebo.xacro" />
     <xacro:include filename="gripper.xacro" />
+    <xacro:include filename="camera.xacro" />
 </robot>

File: src/robot_description/urdf/gripper.xacro (robot description, xacro)
@@ -88,12 +88,4 @@
         <child link="gripper_base" />
     </joint>
-    <!-- gripper left jaw → gripper base -->
-    <joint name="right_jaw_to_gripper_base" type="prismatic">
-        <origin xyz="0 0 0.1358" rpy="1.5708 0 0" />
-        <parent link="gripper_base" />
-        <child link="gripper_left_jaw" />
-        <axis xyz="0 0 1" />
-        <limit lower="0" upper="0.035" effort="10" velocity="1" />
-    </joint>
     <!-- gripper right jaw → gripper base -->
     <joint name="left_jaw_to_gripper_base" type="prismatic">
@@ -104,3 +96,12 @@
         <limit lower="-0.035" upper="0" effort="10" velocity="1" />
     </joint>
+    <!-- gripper right jaw → gripper base -->
+    <joint name="right_jaw_to_gripper_base" type="prismatic">
+        <origin xyz="0 0 0.1358" rpy="1.5708 0 0" />
+        <parent link="gripper_base" />
+        <child link="gripper_left_jaw" />
+        <axis xyz="0 0 1" />
+        <mimic joint="left_jaw_to_gripper_base" multiplier="-1.0" offset="0.0" />
+        <limit lower="-0.001" upper="0.035" effort="10" velocity="1" />
+    </joint>
 </robot>

File: src/robot_moveit_config/config/piper_arm.ros2_control.xacro (robot description, xacro)
@@ -51,4 +51,11 @@
                 <state_interface name="velocity"/>
             </joint>
+            <joint name="left_jaw_to_gripper_base">
+                <command_interface name="position"/>
+                <state_interface name="position">
+                  <param name="initial_value">${initial_positions['left_jaw_to_gripper_base']}</param>
+                </state_interface>
+                <state_interface name="velocity"/>
+            </joint>
         </ros2_control>
         <gazebo>
